Commit message: '前端任务阶段2半'

File: frontend/ur5-control/public/models/ur5.urdf (robot description, URDF)
Before this commit: robot ur5_robot, 11 links, 10 joints
Links:
- link base_link_inertia: geometry collision mesh filename=./collision/base.stl; visual mesh filename=./visual/base.dae
- link forearm_link: geometry collision mesh filename=./collision/forearm.stl; visual mesh filename=./visual/forearm.dae
- link shoulder_link: geometry collision mesh filename=./collision/shoulder.stl; visual mesh filename=./visual/shoulder.dae
- link upper_arm_link: geometry collision mesh filename=./collision/upperarm.stl; visual mesh filename=./visual/upperarm.dae
- link wrist_1_link: geometry collision mesh filename=./collision/wrist1.stl; visual mesh filename=./visual/wrist1.dae
- link wrist_2_link: geometry collision mesh filename=./collision/wrist2.stl; visual mesh filename=./visual/wrist2.dae
- link wrist_3_link: geometry collision mesh filename=./collision/wrist3.stl; visual mesh filename=./visual/wrist3.dae

Commit message: feat: add robotiq gripper assets and simulation control

File: frontend/ur5-control/public/models/ur5.urdf (robot description, URDF)
Before this commit: robot ur5_robot, 11 links, 10 joints
Links:
- added link left_coupler_link, mass 0.0140974; collision mesh filename=robotiq_2f85_v4/coupler.stl; visual mesh filename=robotiq_2f85_v4/coupler.stl
- added link left_driver_link, mass 0.00899563; collision mesh filename=robotiq_2f85_v4/driver.stl; visual mesh filename=robotiq_2f85_v4/driver.stl
- added link left_follower_link, mass 0.0125222; collision mesh filename=robotiq_2f85_v4/follower.stl; collision mesh filename=robotiq_2f85_v4/tongue.stl
- added link left_pad_link, mass 0.002; collision mesh filename=robotiq_2f85_v4/pad.stl; visual mesh filename=robotiq_2f85_v4/pad.stl
- added link left_spring_link, mass 0.0221642; collision mesh filename=robotiq_2f85_v4/spring_link.stl; visual mesh filename=robotiq_2f85_v4/spring_link.stl
- added link right_coupler_link, mass 0.0140974; collision mesh filename=robotiq_2f85_v4/coupler.stl; visual mesh filename=robotiq_2f85_v4/coupler.stl
- added link right_driver_link, mass 0.00899563; collision mesh filename=robotiq_2f85_v4/driver.stl; visual mesh filename=robotiq_2f85_v4/driver.stl
- added link right_follower_link, mass 0.0125222; collision mesh filename=robotiq_2f85_v4/follower.stl; collision mesh filename=robotiq_2f85_v4/tongue.stl
- added link right_pad_link, mass 0.002; collision mesh filename=robotiq_2f85_v4/pad.stl; visual mesh filename=robotiq_2f85_v4/pad.stl
- added link right_spring_link, mass 0.0221642; collision mesh filename=robotiq_2f85_v4/spring_link.stl; visual mesh filename=robotiq_2f85_v4/spring_link.stl
- added link robotiq_base_link, mass 0.777441; collision mesh filename=robotiq_2f85_v4/base.stl; collision mesh filename=robotiq_2f85_v4/base_coupling.stl
- link base_link_inertia: geometry collision mesh filename=collision/base.stl; visual mesh filename=visual/base.dae
- link forearm_link: geometry collision mesh filename=collision/forearm.stl; visual mesh filename=visual/forearm.dae
- link shoulder_link: geometry collision mesh filename=collision/shoulder.stl; visual mesh filename=visual/shoulder.dae
- link upper_arm_link: geometry collision mesh filename=collision/upperarm.stl; visual mesh filename=visual/upperarm.dae
- link wrist_1_link: geometry collision mesh filename=collision/wrist1.stl; visual mesh filename=visual/wrist1.dae
- link wrist_2_link: geometry collision mesh filename=collision/wrist2.stl; visual mesh filename=visual/wrist2.dae
- link wrist_3_link: geometry collision mesh filename=collision/wrist3.stl; visual mesh filename=visual/wrist3.dae
Joints:
- added joint left_driver-left_coupler: type fixed, parent left_driver_link, child left_coupler_link, origin xyz=-0.0314249 0.00453223 -0.0102 rpy=0 0 0
- added joint left_driver_joint: type revolute, parent robotiq_base_link, child left_driver_link, origin xyz=-0.0306011 0.00475 0.0657045 rpy=-1.5707963267948966 0 0, axis 0 0 1, limit lower=0.0 upper=0.9 effort=10.0 velocity=2.0
- added joint left_follower-left_pad: type fixed, parent left_follower_link, child left_pad_link, origin xyz=-0.0377897 -0.103916 -0.0091 rpy=-1.5707963267948966 0 0
- added joint left_follower_joint: type revolute, parent left_spring_link, child left_follower_link, origin xyz=-0.0382079 -0.0425003 0.00295 rpy=3.141592653589793 0 0, axis 0 0 1, limit lower=-0.872664 upper=0.9 effort=10.0 velocity=2.0
- added joint left_spring_link_joint: type revolute, parent robotiq_base_link, child left_spring_link, origin xyz=-0.0127 -0.012 0.07222 rpy=-1.5707963267948966 0 0, axis 0 0 1, limit lower=-0.29670597283 upper=0.9 effort=10.0 velocity=2.0
- added joint right_driver-right_coupler: type fixed, parent right_driver_link, child right_coupler_link, origin xyz=-0.0314249 0.00453223 -0.0102 rpy=0 0 0
- added joint right_driver_joint: type revolute, parent robotiq_base_link, child right_driver_link, origin xyz=0.0306011 -0.00475 0.0657045 rpy=-1.5707963267948966 0 3.141592653589793, axis 0 0 1, limit lower=0.0 upper=0.9 effort=10.0 velocity=2.0
- added joint right_follower-right_pad: type fixed, parent right_follower_link, child right_pad_link, origin xyz=-0.0377897 -0.103916 -0.0091 rpy=-1.5707963267948966 0 0
- added joint right_follower_joint: type revolute, parent right_spring_link, child right_follower_link, origin xyz=-0.0382079 -0.0425003 0.00295 rpy=3.141592653589793 0 0, axis 0 0 1, limit lower=-0.872664 upper=0.9 effort=10.0 velocity=2.0
- added joint right_spring_link_joint: type revolute, parent robotiq_base_link, child right_spring_link, origin xyz=0.0127 0.012 0.07222 rpy=-1.5707963267948966 0 3.141592653589793, axis 0 0 1, limit lower=-0.29670597283 upper=0.9 effort=10.0 velocity=2.0
- added joint tool0-robotiq_base: type fixed, parent tool0, child robotiq_base_link, origin xyz=0 0 0 rpy=0 0 0

File: frontend/ur5/ur5.urdf (robot description, URDF)
Before this commit: robot ur5_robot, 11 links, 10 joints
Links:
- added link left_coupler_link, mass 0.0140974; collision mesh filename=robotiq_2f85_v4/coupler.stl; visual mesh filename=robotiq_2f85_v4/coupler.stl
- added link left_driver_link, mass 0.00899563; collision mesh filename=robotiq_2f85_v4/driver.stl; visual mesh filename=robotiq_2f85_v4/driver.stl
- added link left_follower_link, mass 0.0125222; collision mesh filename=robotiq_2f85_v4/follower.stl; collision mesh filename=robotiq_2f85_v4/tongue.stl
- added link left_pad_link, mass 0.002; collision mesh filename=robotiq_2f85_v4/pad.stl; visual mesh filename=robotiq_2f85_v4/pad.stl
- added link left_spring_link, mass 0.0221642; collision mesh filename=robotiq_2f85_v4/spring_link.stl; visual mesh filename=robotiq_2f85_v4/spring_link.stl
- added link right_coupler_link, mass 0.0140974; collision mesh filename=robotiq_2f85_v4/coupler.stl; visual mesh filename=robotiq_2f85_v4/coupler.stl
- added link right_driver_link, mass 0.00899563; collision mesh filename=robotiq_2f85_v4/driver.stl; visual mesh filename=robotiq_2f85_v4/driver.stl
- added link right_follower_link, mass 0.0125222; collision mesh filename=robotiq_2f85_v4/follower.stl; collision mesh filename=robotiq_2f85_v4/tongue.stl
- added link right_pad_link, mass 0.002; collision mesh filename=robotiq_2f85_v4/pad.stl; visual mesh filename=robotiq_2f85_v4/pad.stl
- added link right_spring_link, mass 0.0221642; collision mesh filename=robotiq_2f85_v4/spring_link.stl; visual mesh filename=robotiq_2f85_v4/spring_link.stl
- added link robotiq_base_link, mass 0.777441; collision mesh filename=robotiq_2f85_v4/base.stl; collision mesh filename=robotiq_2f85_v4/base_coupling.stl
- link base_link_inertia: geometry collision mesh filename=collision/base.stl; visual mesh filename=visual/base.dae
- link forearm_link: geometry collision mesh filename=collision/forearm.stl; visual mesh filename=visual/forearm.dae
- link shoulder_link: geometry collision mesh filename=collision/shoulder.stl; visual mesh filename=visual/shoulder.dae
- link upper_arm_link: geometry collision mesh filename=collision/upperarm.stl; visual mesh filename=visual/upperarm.dae
- link wrist_1_link: geometry collision mesh filename=collision/wrist1.stl; visual mesh filename=visual/wrist1.dae
- link wrist_2_link: geometry collision mesh filename=collision/wrist2.stl; visual mesh filename=visual/wrist2.dae
- link wrist_3_link: geometry collision mesh filename=collision/wrist3.stl; visual mesh filename=visual/wrist3.dae
Joints:
- added joint left_driver-left_coupler: type fixed, parent left_driver_link, child left_coupler_link, origin xyz=-0.0314249 0.00453223 -0.0102 rpy=0 0 0
- added joint left_driver_joint: type revolute, parent robotiq_base_link, child left_driver_link, origin xyz=-0.0306011 0.00475 0.0657045 rpy=-1.5707963267948966 0 0, axis 0 0 1, limit lower=0.0 upper=0.9 effort=10.0 velocity=2.0
- added joint left_follower-left_pad: type fixed, parent left_follower_link, child left_pad_link, origin xyz=-0.0377897 -0.103916 -0.0091 rpy=-1.5707963267948966 0 0
- added joint left_follower_joint: type revolute, parent left_spring_link, child left_follower_link, origin xyz=-0.0382079 -0.0425003 0.00295 rpy=3.141592653589793 0 0, axis 0 0 1, limit lower=-0.872664 upper=0.9 effort=10.0 velocity=2.0
- added joint left_spring_link_joint: type revolute, parent robotiq_base_link, child left_spring_link, origin xyz=-0.0127 -0.012 0.07222 rpy=-1.5707963267948966 0 0, axis 0 0 1, limit lower=-0.29670597283 upper=0.9 effort=10.0 velocity=2.0
- added joint right_driver-right_coupler: type fixed, parent right_driver_link, child right_coupler_link, origin xyz=-0.0314249 0.00453223 -0.0102 rpy=0 0 0
- added joint right_driver_joint: type revolute, parent robotiq_base_link, child right_driver_link, origin xyz=0.0306011 -0.00475 0.0657045 rpy=-1.5707963267948966 0 3.141592653589793, axis 0 0 1, limit lower=0.0 upper=0.9 effort=10.0 velocity=2.0
- added joint right_follower-right_pad: type fixed, parent right_follower_link, child right_pad_link, origin xyz=-0.0377897 -0.103916 -0.0091 rpy=-1.5707963267948966 0 0
- added joint right_follower_joint: type revolute, parent right_spring_link, child right_follower_link, origin xyz=-0.0382079 -0.0425003 0.00295 rpy=3.141592653589793 0 0, axis 0 0 1, limit lower=-0.872664 upper=0.9 effort=10.0 velocity=2.0
- added joint right_spring_link_joint: type revolute, parent robotiq_base_link, child right_spring_link, origin xyz=0.0127 0.012 0.07222 rpy=-1.5707963267948966 0 3.141592653589793, axis 0 0 1, limit lower=-0.29670597283 upper=0.9 effort=10.0 velocity=2.0
- added joint tool0-robotiq_base: type fixed, parent tool0, child robotiq_base_link, origin xyz=0 0 0 rpy=0 0 0
